File: hardware/md/1.10/retrolink.kicad_pcb (KiCad board)
At the start: 2 copper layers, 43 x 28 mm, 5 parts, among them J1 DE9_Socket, J2 DE9_Pins

Commit message: hardware fix. v1.10 MD
Routing:
- net GND: track 0.00 -> 14.5 mm, vias 2 -> 3
Changed lines of the file:
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@@
+	)
+	(via
+		(at 129.3 94.52)
+		(size 0.8)
+		(drill 0.4)
+		(layers "F.Cu" "B.Cu")
+		(net "GND")
 	)
 	(via
@@
 		(net "GND")
 	)
+	(segment
+		(start 142.9 92.4)
+		(end 140.78 94.52)
+		(width 0.3)
+		(layer "B.Cu")
+		(net "GND")
+	)
+	(segment
+		(start 140.78 94.52)
+		(end 129.3 94.52)
+		(width 0.3)
+		(layer "B.Cu")
+		(net "GND")
+	)
